Commit message: Phase 6: Fix bread_v41 collision mesh + cluster validation PASS
- Centered visual mesh at origin (182 verts, 360 faces)
- Generated dedicated collision box (8 verts, 12 tris, centered)
- Updated URDF: separate visual/collision meshes, origins at (0,0,0)
- Cluster validation: stable physics, zero drift, no sinking
- Added collision fix script and render attempt scripts
- Documented cluster validation results

Co-Authored-By: Claude Fable 5 <noreply@anthropic.com>

File: experiments/2026-07-04_obj_recon_bread/models/bread_v41.urdf (robot description, URDF)
Before this commit: robot bread, 1 links, 0 joints
Links:
- link base_link: geometry collision mesh filename=bread_v41_collision.obj scale=1.0 1.0 1.0; visual mesh filename=bread_v41.obj scale=1.0 1.0 1.0
