Commit message: task3: fix stale metadata, realistic masses, pipette Y-dim, geometry reports
- Fix object_meta.json: updated face counts and masses to match actual meshes
- Fix pipette Y dimension: 0.104m → 0.020m (422% deviation corrected)
- Fix masses: bread=0.40, pipette=0.15, drinks=0.55 kg (realistic values)
- Remove stale geometry_check_collision.txt files (referenced deleted box meshes)
- Regenerate geometry_quality_report.txt with explicit manifold checks
- Update isaacgym_validation_summary.json (was incorrectly showing failed_local_env)
- All 4 URDFs updated with correct mass/inertia, re-validated: 4/4 PASS

File: runs/object_asset_v1/bread/asset/object.urdf (robot description, URDF)
Before this commit: robot bread, 1 links, 0 joints
Links:
- link base_link: mass 0.0775 -> 0.4000

File: runs/object_asset_v1/drink_ad/asset/object.urdf (robot description, URDF)
Before this commit: robot drink_ad, 1 links, 0 joints
Links:
- link base_link: mass 1.4695 -> 0.5500

File: runs/object_asset_v1/drink_yykx/asset/object.urdf (robot description, URDF)
Before this commit: robot drink_yykx, 1 links, 0 joints
Links:
- link base_link: mass 0.8571 -> 0.5500

File: runs/object_asset_v1/pipette/asset/object.urdf (robot description, URDF)
Before this commit: robot pipette, 1 links, 0 joints
Links:
- link base_link: mass 1.2116 -> 0.1500

Commit message: task3: advanced 3D reconstruction V2 — object-specific modeling
- Drinks: cylinder mesh (circle-fit from top mask, height from side mask)
  drink_ad: r=49mm h=91mm 0.68kg, drink_yykx: r=49mm h=101mm 0.76kg
- Bread: organic extrusion (top contour + tapered height profile)
  1781v 3288f, rounded organic shape
- Pipette: variable-section extrusion (top contour + side width profile)
  128v, mass 0.59kg
- Fixed: cylinder face winding (volume was negative)
- All IsaacGym videos regenerated with new models (48 MP4s)
- Backups: visual_mesh_backup.obj

File: runs/object_asset_v1/bread/asset/object.urdf (robot description, URDF)
Before this commit: robot bread, 1 links, 0 joints
Links:
- link base_link: mass 0.4000 -> 0.1016

File: runs/object_asset_v1/drink_ad/asset/object.urdf (robot description, URDF)
Before this commit: robot drink_ad, 1 links, 0 joints
Links:
- link base_link: mass 0.5500 -> 0.6823

File: runs/object_asset_v1/drink_yykx/asset/object.urdf (robot description, URDF)
Before this commit: robot drink_yykx, 1 links, 0 joints
Links:
- link base_link: mass 0.5500 -> 0.7616

File: runs/object_asset_v1/pipette/asset/object.urdf (robot description, URDF)
Before this commit: robot pipette, 1 links, 0 joints
Links:
- link base_link: mass 0.1500 -> 0.5898

Commit message: task3: advanced 3D reconstruction V3 — fix remaining limitations
- Bread: watertight organic mesh with top/bottom caps (1128v, 2252f, wt=True)
- Pipette: multi-slice cross-section from top contour + side thickness (46v, 86f)
- Drinks: cylinder models with correct face winding
- Fixed: trimesh.repair.broken_faces returns ndarray, handle correctly
- All 48 IsaacGym videos regenerated

File: runs/object_asset_v1/bread/asset/object.urdf (robot description, URDF)
Before this commit: robot bread, 1 links, 0 joints
Links:
- link base_link: mass 0.1016 -> 0.0698

File: runs/object_asset_v1/drink_ad/asset/object.urdf (robot description, URDF)
Before this commit: robot drink_ad, 1 links, 0 joints
Links:
- link base_link: mass 0.6823 -> 0.3147

File: runs/object_asset_v1/drink_yykx/asset/object.urdf (robot description, URDF)
Before this commit: robot drink_yykx, 1 links, 0 joints
Links:
- link base_link: mass 0.7616 -> 0.2775

File: runs/object_asset_v1/pipette/asset/object.urdf (robot description, URDF)
Before this commit: robot pipette, 1 links, 0 joints
Links:
- link base_link: mass 0.5898 -> 0.7171

Commit message: task3: 3D model quality upgrade — vertex colors + hi-res reconstruction
Reconstruction quality:
- Contour points: 200→300, Z-slices: 8→16
- bread: 588→1116 faces, pipette: 3196→9596 faces (3x denser)
- drink_ad: 460→988 faces, drink_yykx: 284→636 faces

Vertex colors:
- 100% vertices colored from 3 camera video frames (top+side_1+side_2)
- Multi-view color blending for complete coverage
- Saved as textured_mesh.obj and textured_mesh.ply

Geometry:
- All 4 objects watertight + correct extents
- Drinks: cylindrical symmetry enforced (0.07×0.07×0.20m)
- Pipette: Y=0.02m correct

Validation: 4/4 IsaacGym PASS
Renders: 20 colored renders (38-192KB each)

File: runs/object_asset_v1/bread/asset/object.urdf (robot description, URDF)
Before this commit: robot bread, 1 links, 0 joints
Links:
- link base_link: mass 0.0698 -> 0.4000

File: runs/object_asset_v1/drink_ad/asset/object.urdf (robot description, URDF)
Before this commit: robot drink_ad, 1 links, 0 joints
Links:
- link base_link: mass 0.3147 -> 0.5500

File: runs/object_asset_v1/drink_yykx/asset/object.urdf (robot description, URDF)
Before this commit: robot drink_yykx, 1 links, 0 joints
Links:
- link base_link: mass 0.2775 -> 0.5500

File: runs/object_asset_v1/pipette/asset/object.urdf (robot description, URDF)
Before this commit: robot pipette, 1 links, 0 joints
Links:
- link base_link: mass 0.7171 -> 0.1500

Commit message: task3: upgrade object reconstruction assets

File: runs/object_asset_v1/bread/asset/object.urdf (robot description, URDF)
Before this commit: robot bread, 1 links, 0 joints
Links:
- link base_link: mass 0.4000 -> 0.076000

File: runs/object_asset_v1/drink_ad/asset/object.urdf (robot description, URDF)
Before this commit: robot drink_ad, 1 links, 0 joints
Links:
- link base_link: mass 0.5500 -> 0.622000

File: runs/object_asset_v1/drink_yykx/asset/object.urdf (robot description, URDF)
Before this commit: robot drink_yykx, 1 links, 0 joints
Links:
- link base_link: mass 0.5500 -> 0.353000

File: runs/object_asset_v1/pipette/asset/object.urdf (robot description, URDF)
Before this commit: robot pipette, 1 links, 0 joints
Links:
- link base_link: mass 0.1500 -> 0.180000
